Commit message: Update vlp16-imu.urdf
removing comments and changing link names

File: cartographer_ros/urdf/vlp16-imu.urdf (robot description, URDF)
Before this commit: robot cartographer_backpack_3d, 3 links, 2 joints
Links:
- removed link horizontal_vlp16_link
- removed link imu_link
- added link imu; visual box size=0.06 0.04 0.02
- added link velodyne; visual cylinder length=0.07 radius=0.05
Joints:
- removed joint horizontal_vlp16_link_joint
- removed joint imu_link_joint
- added joint imu_joint: type fixed, parent base_link, child imu, origin xyz=0 0 0 rpy=3.1416 0 0
- added joint velodyne_joint: type fixed, parent base_link, child velodyne, origin xyz=0.01 0. 0.19 rpy=0. -0.1745 3.1416
